Commit message: Mk0 got a bit of a platform boost because it was hard to get stuff inside.

File: mk0_description/urdf/sensors/ydlidar.urdf.xacro (robot description, xacro)
@@ -29,5 +29,5 @@
       <parent link="${parent}" />
       <child link="lidar_link" />
-      <origin xyz="0.12 0 0.215" rpy="0 0 0" />
+      <origin xyz="0.12 0 0.248" rpy="0 0 0" />
     </joint>
     <!-- simulation sensor -->

File: mk0_description/urdf/stacks/hexagons.urdf.xacro (robot description, xacro)
@@ -153,6 +153,11 @@
     <xacro:stack_middle_pole parent="${parent}" number="2" x_loc="-0.0381" y_loc="0.1505" z_loc="0.1640" />
     <xacro:stack_middle_pole parent="${parent}" number="3" x_loc="-0.0381" y_loc="-0.1505" z_loc="0.1640" />
+    <xacro:stack_middle_pole parent="${parent}" number="4" x_loc="0.0381" y_loc="0.1505" z_loc="0.206" />
+    <xacro:stack_middle_pole parent="${parent}" number="5" x_loc="0.0381" y_loc="-0.1505" z_loc="0.2060" />
+    <xacro:stack_middle_pole parent="${parent}" number="6" x_loc="-0.0381" y_loc="0.1505" z_loc="0.2060" />
+    <xacro:stack_middle_pole parent="${parent}" number="7" x_loc="-0.0381" y_loc="-0.1505" z_loc="0.2060" />
     <joint name="plate_middle_joint" type="fixed">
-      <origin xyz="-0.01364 0.0 0.1874" rpy="0 0 0" />
+      <origin xyz="-0.01364 0.0 0.2240" rpy="0 0 0" />
+      <!-- <origin xyz="-0.01364 0.0 0.1874" rpy="0 0 0" /> -->
       <parent link="${parent}" />
       <child link="plate_middle_link" />

Commit message: i dont know whats going on. xacro -> urdf -> sdf?? collision tags on ydlidar and hexagons have been the things breaking the gazebo simulation. removing collision tag sfrom the ydlidar and hexagons fixes this and allows me to control... I'm not entirely sure why this is, but this whole thing is kinda frankensteined together.. Big progress figuring it out though. I'll ask on discord and maybe askgazebo and see if theres any input there. Since i dont need the upper body collision though i think this is fine for now. cant wait for that one to bite me. Modified simu bringup to help in fixing this in the mean time, will change it back once its all good.
real log:
Changed simu bringup to help debug.
removed collision flags from ydlidar and hexagons xacro files.
fixed ekf in gazebo_display.launch.

File: mk0_description/urdf/sensors/ydlidar.urdf.xacro (robot description, xacro)
@@ -13,10 +13,10 @@
         <inertia ixx="0.001" ixy="0" ixz="0" iyy="0.001" iyz="0" izz="0.001" />
       </inertial>
-      <collision>
+      <!-- <collision>
         <origin xyz="0 0 0" rpy="0 0 0" />
         <geometry>
           <cylinder radius="${x2l_radius}" length="${x2l_height}" />
         </geometry>
-      </collision>
+      </collision> -->
       <visual>
         <origin xyz="0 0 0" rpy="0 0 0" />

File: mk0_description/urdf/stacks/hexagons.urdf.xacro (robot description, xacro)
@@ -22,10 +22,10 @@
         </geometry>
       </visual>
-      <collision>
+      <!-- <collision>
         <origin xyz="0 0 0" rpy="0 0 0" />
         <geometry>
           <cylinder length="0.0492" radius="0.006" />
         </geometry>
-      </collision>
+      </collision> -->
       <inertial>
         <mass value="0.008" />
@@ -48,10 +48,10 @@
         </geometry>
       </visual>
-      <collision>
+      <!-- <collision>
         <origin xyz="0 0 0" rpy="0 0 0" />
         <geometry>
           <cylinder length="0.0608" radius="0.006" />
         </geometry>
-      </collision>
+      </collision> -->
       <inertial>
         <mass value="0.012" />
@@ -74,10 +74,10 @@
         </geometry>
       </visual>
-      <collision>
+      <!-- <collision>
         <origin xyz="0 0 0" rpy="0 0 0" />
         <geometry>
           <cylinder length="0.2032" radius="0.006" />
         </geometry>
-      </collision>
+      </collision> -->
       <inertial>
         <mass value="0.060" />
@@ -100,10 +100,10 @@
         </geometry>
       </visual>
-      <collision>
+      <!-- <collision>
         <origin xyz="0 0 0" rpy="0 0 0" />
         <geometry>
           <cylinder length="0.0936" radius="0.006" />
         </geometry>
-      </collision>
+      </collision> -->
       <inertial>
         <mass value="0.020" />
@@ -137,10 +137,10 @@
         </geometry>
       </visual>
-      <collision>
+      <!-- <collision>
         <origin xyz="-0.02364 0 0" rpy="0 0 0" />
         <geometry>
           <cylinder length="0.006" radius="0.170" />
         </geometry>
-      </collision>
+      </collision> -->
       <inertial>
         <mass value="0.520" />
@@ -170,10 +170,10 @@
         </geometry>
       </visual>
-      <collision>
+      <!-- <collision>
         <origin xyz="0.01364 0.0 0.0" rpy="0 0 0" />
         <geometry>
           <mesh filename="file://$(find mk0_description)/meshes/stacks/hexagons/plate_simple.stl" scale="${M_SCALE} ${M_SCALE} ${M_SCALE}" />
         </geometry>
-      </collision>
+      </collision> -->
       <inertial>
         <mass value="0.520" />
